Commit message: Updated with teleop_twist_keyboard

File: src/Marjanator_description/urdf/materials.xacro (robot description, xacro)
@@ -1,5 +1,5 @@
 <?xml version="1.0" ?>
 <robot name="Marjanator" xmlns:xacro="http://www.ros.org/wiki/xacro" >
-<material name="acrylics">
+<material name="acrylic">
   <color rgba="0.700 0.700 0.700 1.000"/>
 </material>
